File: project_files/rev3/project_rev3/controller.kicad_sch (KiCad schematic)
At the start: 25 parts, among them J8 USB_C_Receptacle_16P, SW1 JS102011SAQN, U5 ESP32-S3-WROOM-1-N16R8, U6 AZ1117CH-3.3

Commit message: added labels to rev3 sch and pcb
Other:
- note added: "BOOT button - hold boot while flashing to upload"
- note added: "The files for these buttons are insane- the models don't reflect the actual parts. Change this."
- note added: "USB C and Power_PROG are for programming only. SW1 is dip switch to switch power from the functioning FLOPS system to USB. It has its own LDO to simplify things."
Changed lines of the file:
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@@
 	)
 	(rectangle
-		(start 281.686 40.132)
-		(end 326.136 128.778)
+		(start 17.78 76.2)
+		(end 173.99 161.29)
+		(stroke
+			(width 0)
+			(type default)
+		)
+		(fill
+			(type none)
+		)
+	)
+	(rectangle
+		(start 188.976 62.992)
+		(end 254 154.94)
 		(stroke
 			(width 0.254)
@@
 	(text "Controller\n"
 		(exclude_from_sim no)
-		(at 288.29 41.91 0)
+		(at 196.342 59.944 0)
 		(effects
 			(font
@@
 			)
 		)
+	)
+	(text "The files for these buttons are insane- the models don't reflect\nthe actual parts. Change this.\n"
+		(exclude_from_sim no)
+		(at 83.312 25.146 0)
+		(effects
+			(font
+				(size 1.27 1.27)
+			)
+		)
+	)
+	(text "USB C and Power_PROG are for programming only.\nSW1 is dip switch to switch power from the functioning\nFLOPS system to USB. It has its own LDO to simplify things."
+		(exclude_from_sim no)
+		(at 49.276 83.312 0)
+		(effects
+			(font
+				(size 1.27 1.27)
+			)
+		)
+	)
+	(text "BOOT button - hold boot while flashing to upload"
+		(exclude_from_sim no)
+		(at 43.942 65.278 0)
+		(effects
+			(font
+				(size 1.27 1.27)
+			)
+		)
