File: project_files/rev3/project_rev3/project_rev3.kicad_sch (KiCad schematic)
At the start: 31 parts, among them J1 Barrel_Jack, J2 Conn_01x04, J3 Conn_01x02, J4 Conn_01x02, J5 Conn_01x02, J6 Conn_01x02, J7 Conn_01x02, Q1 BSS816NWH6327XTSA1, Q2 S8550, U1 HX711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

Commit message: added labels to rev3 sch and pcb
Changed lines of the file:
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@@
 	)
 	(rectangle
-		(start 146.05 -24.13)
-		(end 236.22 10.16)
+		(start 151.13 24.13)
+		(end 273.05 69.85)
 		(stroke
 			(width 0.254)
@@
 		)
 		(instances
-			(project "project1"
+			(project "project_rev3"
 				(path "/2c76aad2-f58e-4a51-9b78-5834a8cd02ae"
 					(page "2")
