File: project_files/rev3/project_rev3/project_rev3.kicad_sch (KiCad schematic)
At the start: 28 parts, among them J1 Barrel_Jack, J2 Conn_01x04, J3 Conn_01x02, J4 Conn_01x02, J5 Conn_01x02, J6 Conn_01x02, J7 Conn_01x02, Q1 NMOS, Q2 S8550, U1 HX711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

Commit message: rev3 schematic and layout (#32)
* renamed project to current rev. each future rev will get it's own copy in project directory. each rev will not be touched once it has been committed and another rev is being worked on. Added update sch and pcb.

* added labels to rev3 sch and pcb

* printed pdf of sch and pcb

* moved something
Parts:
- removed R10, R11, R8, R9: 0603, Resistor_SMD:R_0201_0603Metric, symbol Device:R_Small
- removed U2: ESP32-WROOM-32, RF_Module:ESP32-WROOM-32, symbol RF_Module:ESP32-WROOM-32
- removed U6: 74LS21, Package_SO:SO-14_5.3x10.2mm_P1.27mm, symbol 74xx:74LS21
- added C5, C7: 10uF, Capacitor_SMD:C_0603_1608Metric_Pad1.08x0.95mm_HandSolder, symbol Device:C_Small
- added C6, C8: 0.1uF, Capacitor_SMD:C_0603_1608Metric_Pad1.08x0.95mm_HandSolder, symbol Device:C_Small
- added RV1, RV2, RV3, RV4: 100k Trim Pot, Potentiometer_SMD:Potentiometer_Bourns_3314G_Vertical, symbol Device:R_Potentiometer_Trim
- added U2: 74LS21, Package_SO:SOIC-14_3.9x8.7mm_P1.27mm, symbol 74xx:74LS21
- C1: value 0603 -> 10uF; footprint Capacitor_SMD:C_0201_0603Metric -> Capacitor_SMD:C_0603_1608Metric_Pad1.08x0.95mm_HandSolder
- C2, C3, C4: value 0603 -> 0.1uF; footprint Capacitor_SMD:C_0201_0603Metric -> Capacitor_SMD:C_0603_1608Metric_Pad1.08x0.95mm_HandSolder
- J1: symbol Connector:Barrel_Jack -> Connector:Barrel_Jack_Switch_Pin3Ring
- J3, J4, J5, J6, J7: footprint Connector_JST:JST_XA_S02B-XASK-1_1x02_P2.50mm_Horizontal -> Connector_JST:JST_XA_S02B-XASK-1N-BN_1x02_P2.50mm_Horizontal
- Q1: value NMOS -> BSS816NWH6327XTSA1
- R1: value 0603 -> 100; footprint (none) -> Resistor_SMD:R_0603_1608Metric_Pad0.98x0.95mm_HandSolder
- R3: value 0603 -> 10k; footprint (none) -> Resistor_SMD:R_0603_1608Metric_Pad0.98x0.95mm_HandSolder
- R4: value 0603 -> 20k; footprint Resistor_SMD:R_0201_0603Metric -> Resistor_SMD:R_0603_1608Metric_Pad0.98x0.95mm_HandSolder
- R5: value 0603 -> 8.2k; footprint Resistor_SMD:R_0201_0603Metric -> Resistor_SMD:R_0603_1608Metric_Pad0.98x0.95mm_HandSolder
- R6, R7: value 0603 -> 100; footprint Resistor_SMD:R_0201_0603Metric -> Resistor_SMD:R_0603_1608Metric_Pad0.98x0.95mm_HandSolder
- U3: footprint Package_TO_SOT_SMD:SOT-223 -> Package_TO_SOT_SMD:SOT-223-3_TabPin2
Connections:
- net +5 is gone; now on net +5V_WALL: J3.2 (Pin_2), J4.2 (Pin_2), J5.2 (Pin_2), J6.2 (Pin_2)
- net GND: now also J1.3, C5.2, C6.2, C7.2, C8.2, RV1.3, RV2.3, RV3.3, RV4.3, U2.7 (GND)
- net at U4.5 (+): now also RV2.2; no longer J4.1 (Pin_1)
- net at U4.6 (-), U4.7: now also U2.2
- net at J5.1 (Pin_1): now also RV3.1; no longer U4.10 (+)
- net NFET_3.3V: now reaches Q1.3 (S)
- net GPIO_36: now reaches U1.11 (PD_SCK)
- net GPIO_35: now reaches U1.12 (DOUT)
- net at U4.8, U4.9 (-): now also U2.4
- net +5V_WALL: now reaches J7.2 (Pin_2), U3.3 (VI)
- net +5V_WALL: now also U4.4 (V+), C5.1, C6.1, U2.14 (VCC)
- net at U4.1, U4.2 (-): now also U2.1
- net at U4.13 (-), U4.14: now also U2.5
- net at R1.1: now also U2.6
- net at J3.1 (Pin_1): now also RV1.1; no longer U4.3 (+)
- net at J6.1 (Pin_1): now also RV4.1; no longer U4.12 (+)
- net +3.3V renamed ESP_3.3V
- net ESP_3.3V: no longer Q1.1 (D), U3.2 (VO)
- net +5V: no longer names the net of J1.1, J7.1 (Pin_1)
- net +5V: no longer U4.4 (V+)
- new net: RV3.2, U4.10 (+)
- new net: RV1.2, U4.3 (+)
- new net: RV4.2, U4.12 (+)
- new net: J4.1 (Pin_1), RV2.1
- new net +3.3V_WALL: C7.1, C8.1, Q1.1 (D), U3.2 (VO)
- no-connect marks 0 -> 6
Other:
- added sheet controller (controller.kicad_sch)
- note added: "Power_FLOPS"
- note removed: "Controller"
- note removed: "ESP32 will require additional connections, components, depending on mfg recommendations. Those, also TBD."
- note removed: "NOTE WHILE DOING LAYOUT: Might be worth labeling some of these nets. SMP"
- note removed: "Power"
- note removed: "STILL NEED MOSFET DRIVER SELECTION. TBD."
- title: FOPS -> FLOPS
- moved on the sheet: J3, J7, U3
