File: project_files/real_rev3/project_rev3/project_rev3.kicad_sch (KiCad schematic)
At the start: 34 parts, among them J1 Barrel_Jack, J2 Conn_01x04, J3 Conn_01x02, J4 Conn_01x02, J5 Conn_01x02, J6 Conn_01x02, J7 Conn_01x02, Q1 BSS816NWH6327XTSA1, Q2 S8550, U1 HX711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

Commit message: fucked up a commit, tring to fix
Parts:
- removed R10, R11, R9: 0, Resistor_SMD:R_0603_1608Metric_Pad0.98x0.95mm_HandSolder, symbol Device:R_Small
Connections:
- net +3.3V_WALL: now also Q1.1 (D)
- net NFET_3.3V: now also Q1.3 (S)
- net at R1.2, R3.1: now also Q1.2 (G)
Other:
- moved on the sheet: Q1
