File: project_files/rev4/project_rev4/project_rev4.kicad_sch (KiCad schematic)
At the start: 31 parts, among them J1 Barrel_Jack, J2 Conn_01x04, J3 Conn_01x02, J4 Conn_01x02, J5 Conn_01x02, J6 Conn_01x02, J7 Conn_01x02, Q1 BSS816NWH6327XTSA1, Q2 S8550, U1 HX711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

Commit message: committing update
Parts:
- added R10, R11, R16, R17, R9: 0, Resistor_SMD:R_0603_1608Metric_Pad0.98x0.95mm_HandSolder, symbol Device:R_Small
- RV1, RV2, RV3, RV4: footprint Potentiometer_SMD:Potentiometer_Bourns_3314G_Vertical -> Potentiometer_SMD:Potentiometer_Bourns_TC33X_Vertical
Connections:
- net +3.3V_WALL: now also R9.2
- net ESP_3.3V: now also R11.1; no longer C1.2, Q2.1 (E), U1.1 (VSUP), U1.16 (DVDD)
- net GPIO_35: now also R17.1; no longer U1.12 (DOUT)
- net GPIO_36: now also R16.1; no longer U1.11 (PD_SCK)
- net NFET_3.3V: now also R10.1; no longer Q1.3 (S)
- net AND_OUT: now reaches Q1.2 (G), R1.2, R3.1
- new net: R17.2, U1.12 (DOUT)
- new net: C1.2, Q2.1 (E), R11.2, U1.1 (VSUP), U1.16 (DVDD)
- new net: R16.2, U1.11 (PD_SCK)
- new net: Q1.3 (S), R10.2, R9.1
Other:
- moved on the sheet: Q1
