File: project_files/rev4/project_rev4/project_rev4.kicad_pcb (KiCad board)
At the start: 2 copper layers, 86 x 109 mm, 56 parts, among them J1 Barrel_Jack, J2 Conn_01x04, J3 Conn_01x02, J4 Conn_01x02, J5 Conn_01x02, J6 Conn_01x02, J7 Conn_01x02, J8 USB_C_Receptacle_USB2.0_16P, Q1 BSS816NWH6327XTSA1, Q2 S8550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

Commit message: committing update
Parts:
- added J10: Conn_01x09, Connector_PinHeader_2.54mm:PinHeader_1x09_P2.54mm_Vertical, F.Cu at (120.9, 156.3)
- added J11: Conn_01x10, Connector_PinHeader_2.54mm:PinHeader_1x10_P2.54mm_Vertical, F.Cu at (52.0, 157.1)
- added J12: Conn_01x12, Connector_PinHeader_2.54mm:PinHeader_1x12_P2.54mm_Vertical, F.Cu at (72.9, 134.8)
- added R10: 0, Resistor_SMD:R_0603_1608Metric_Pad0.98x0.95mm_HandSolder, F.Cu at (102.0, 86.4)
- added R11: 0, Resistor_SMD:R_0603_1608Metric_Pad0.98x0.95mm_HandSolder, F.Cu at (69.9, 126.6)
- added R12: 0, Resistor_SMD:R_0603_1608Metric_Pad0.98x0.95mm_HandSolder, F.Cu at (107.0, 117.9)
- added R16: 0, Resistor_SMD:R_0603_1608Metric_Pad0.98x0.95mm_HandSolder, F.Cu at (74.0, 144.9)
- added R17: 0, Resistor_SMD:R_0603_1608Metric_Pad0.98x0.95mm_HandSolder, F.Cu at (74.1, 141.7)
- added R9: 0, Resistor_SMD:R_0603_1608Metric_Pad0.98x0.95mm_HandSolder, F.Cu at (99.9, 75.5)
- RV1, RV2, RV3, RV4: footprint Potentiometer_SMD:Potentiometer_Bourns_3314G_Vertical -> Potentiometer_SMD:Potentiometer_Bourns_TC33X_Vertical
- moved U1 11.5 mm to (66.9, 141.9)
- moved C3 9.21 mm to (60.8, 141.2)
- moved R15 7.73 mm to (110.1, 144.1)
- moved C12 6.64 mm to (113.5, 145.9)
- moved C9 5.40 mm to (121.2, 127.3)
- moved C15 5.40 mm to (114.2, 139.4)
- moved C16 5.40 mm to (114.2, 135.4)
- moved C17 5.40 mm to (109.9, 135.4)
- moved C18 5.40 mm to (109.9, 139.4)
- moved U6 5.40 mm to (111.2, 128.4)
- moved SW2 5.15 mm to (86.5, 124.3)
- moved C1 4.51 mm to (59.5, 123.7)
- moved Q2 4.51 mm to (54.4, 124.6)
- moved C2 4.51 mm to (51.5, 135.5)
- moved C4 4.51 mm to (58.5, 144.7)
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Connections:
- net Net-(Q1-G) renamed /AND_OUT
- C1 pad 2: ESP_3.3V -> Net-(Q2-E)
- Q1 pad 3: NFET_3.3V -> Net-(Q1-S)
- Q2 pad 1: ESP_3.3V -> Net-(Q2-E)
- SW1 pad 3: ESP_3.3V -> Net-(SW1-A)
- U1 pad 1: ESP_3.3V -> Net-(Q2-E)
- U1 pad 11: GPIO_36 -> Net-(U1-PD_SCK)
- U1 pad 12: GPIO_35 -> Net-(U1-DOUT)
- U1 pad 16: ESP_3.3V -> Net-(Q2-E)
- U5 pad 10: unconnected-(U5-GPIO17-Pad10) -> GPIO_17
- U5 pad 11: unconnected-(U5-GPIO18/CLK_OUT3-Pad11) -> GPIO_18
- U5 pad 12: unconnected-(U5-GPIO8-Pad12) -> GPIO_08
- U5 pad 15: unconnected-(U5-GPIO3-Pad15) -> GPIO_03
- U5 pad 16: unconnected-(U5-GPIO46-Pad16) -> GPIO_46
- U5 pad 17: unconnected-(U5-GPIO9-Pad17) -> GPIO_09
- U5 pad 18: unconnected-(U5-GPIO10-Pad18) -> GPIO_10
- U5 pad 19: unconnected-(U5-GPIO11-Pad19) -> GPIO_11
- U5 pad 20: unconnected-(U5-GPIO12-Pad20) -> GPIO_12
- U5 pad 21: unconnected-(U5-GPIO13-Pad21) -> GPIO_13
- U5 pad 22: unconnected-(U5-GPIO14-Pad22) -> GPIO_14
- U5 pad 23: unconnected-(U5-GPIO21-Pad23) -> GPIO_21
- U5 pad 24: unconnected-(U5-GPIO47/SPICLK_P-Pad24) -> GPIO_47
- U5 pad 25: unconnected-(U5-GPIO48/SPICLK_N-Pad25) -> GPIO_48
- U5 pad 26: unconnected-(U5-GPIO45-Pad26) -> GPIO_45
- U5 pad 30: unconnected-(U5-SPIDQS/GPIO37-Pad30) -> GPIO_37
- U5 pad 31: unconnected-(U5-GPIO38-Pad31) -> GPIO_38
- U5 pad 32: unconnected-(U5-MTCK/GPIO39/CLK_OUT3/SUBSPICS1-Pad32) -> GPIO_39
- U5 pad 33: unconnected-(U5-MTDO/GPIO40/CLK_OUT2-Pad33) -> GPIO_40
- U5 pad 34: unconnected-(U5-MTDI/GPIO41/CLK_OUT1-Pad34) -> GPIO_41
- U5 pad 35: unconnected-(U5-MTMS/GPIO42-Pad35) -> GPIO_42
- U5 pad 36: unconnected-(U5-U0RXD/GPIO44/CLK_OUT2-Pad36) -> GPIO_44
- U5 pad 37: unconnected-(U5-U0TXD/GPIO43/CLK_OUT1-Pad37) -> GPIO_43
- U5 pad 38: unconnected-(U5-GPIO2-Pad38) -> GPIO_02
- U5 pad 39: unconnected-(U5-GPIO1-Pad39) -> GPIO_01
- U5 pad 4: unconnected-(U5-GPIO4-Pad4) -> GPIO_04
- U5 pad 5: unconnected-(U5-GPIO5-Pad5) -> GPIO_05
- U5 pad 6: unconnected-(U5-GPIO6-Pad6) -> GPIO_06
- U5 pad 7: unconnected-(U5-GPIO7-Pad7) -> GPIO_07
- U5 pad 8: unconnected-(U5-GPIO15-Pad8) -> GPIO_15
- U5 pad 9: unconnected-(U5-GPIO16-Pad9) -> GPIO_16
Routing:
- net GPIO_37: track 0.00 -> 32.1 mm
- net Net-(Q2-E): track 0.00 -> 30.7 mm
- net GPIO_08: track 0.00 -> 30.0 mm
- net GPIO_38: track 0.00 -> 29.0 mm
- net GPIO_18: track 0.00 -> 26.9 mm
- net GPIO_39: track 0.00 -> 26.0 mm
- net GPIO_17: track 0.00 -> 23.3 mm
- net Net-(SW1-A): track 0.00 -> 23.1 mm
- net GPIO_40: track 0.00 -> 22.9 mm
- net CHIP_PU_EN: track 40.5 -> 63.2 mm
- net GPIO_16: track 0.00 -> 20.3 mm
- net GPIO_41: track 0.00 -> 19.9 mm
- net ESP_3.3V: track 122.4 -> 103.1 mm
- net GPIO_15: track 0.00 -> 17.2 mm
- net GPIO_42: track 0.00 -> 16.7 mm
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
Commit message: final rev4
Other:
- board text added: "Team 09 FLOPS rev4 11/14/2024"
Changed lines of the file:
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@@
+		)
+	)
+	(gr_text "Team 09 \nFLOPS rev4\n11/14/2024\n"
+		(at 99.32 60.33 0)
+		(layer "F.SilkS")
+		(effects
+			(font
+				(size 1.5 1.5)
+				(thickness 0.3)
+				(bold yes)
+			)
+			(justify left bottom)
 		)
 	)
