File: project_files/rev5/project_rev5/controller.kicad_sch (KiCad schematic)
At the start: 35 parts, among them J10 Conn_01x09, J11 Conn_01x10, J12 Conn_01x12, J8 USB_C_Receptacle_USB2.0_16P, SW1 JS102011SAQN, SW2 PTS810 SJM 250 SMTR LFS, SW3 PTS810 SJM 250 SMTR LFS, U5 ESP32-S3-WROOM-1-N16R8, U6 AZ1117CH-3.3

Commit message: pushing final rev5. may god have mercy.
Parts:
- removed SW1: JS102011SAQN, Button_Switch_SMD:SW_SPDT_CK_JS102011SAQN, symbol Switch:SW_SPDT_312
- added SW4: JS102011SAQN, Button_Switch_SMD:SW_SPDT_CK_JS102011SAQN, symbol Switch:SW_Push_SPDT
- added TP_BOOT1, TP_PU_EN1: TestPoint, TestPoint:TestPoint_THTPad_D1.5mm_Drill0.7mm, symbol Connector:TestPoint
Connections:
- net CHIP_PU_EN: now also TP_PU_EN1.1
- net ESP_VCC: now also SW4.2 (B)
- net GPIO0_BOOT: now also TP_BOOT1.1
- net NFET_3.3V: now also SW4.1 (A)
- net at R12.2: now also SW4.3 (C)
Other:
- note added: "All Unused GPIO In Header"
- moved on the sheet: C10, C11, C13, C14, C15, C16, C17, C18, D8, R12, R13, R14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
