File: project_files/rev5/project_rev5/project_rev5.kicad_sch (KiCad schematic)
At the start: 43 parts, among them J1 Barrel_Jack, J2 Conn_01x04, J3 Conn_01x02, J4 Conn_01x02, J5 Conn_01x02, J6 Conn_01x02, J7 Conn_01x02, Q1 BSS816NWH6327XTSA1, Q2 S8550, U1 HX711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

Commit message: pushing final rev5. may god have mercy.
Parts:
- added TP1, TP2: TestPoint, TestPoint:TestPoint_Keystone_5015_Micro-Minature, symbol Connector:TestPoint
- added TP_ADC2, TP_AND1, TP_LCELL_VCC1: TestPoint, TestPoint:TestPoint_THTPad_D1.5mm_Drill0.7mm, symbol Connector:TestPoint
Connections:
- net GND: now also TP1.1, TP2.1
- net at R1.1, U2.6: now also TP_AND1.1
- net at C2.2, J2.1 (Pin_1), Q2.3 (C)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: now also TP_LCELL_VCC1.1
- net at C1.2, Q2.1 (E), R11.2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: now also TP_ADC2.1
Other:
- note removed: "TFT Screen Custom Header/Harness (possible part of actuator- may only be used for WiFi input, may display data)"
- moved on the sheet: H1, H2, H3, H4, U2A
