File: project_files/rev5/project_rev5/project_rev5.kicad_pcb (KiCad board)
At the start: 2 copper layers, 86 x 93 mm, 79 parts, among them J1 Barrel_Jack, J10 Conn_01x09, J11 Conn_01x10, J12 Conn_01x12, J2 Conn_01x04, J3 Conn_01x02, J4 Conn_01x02, J5 Conn_01x02, J6 Conn_01x02, J7 Conn_01x02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

Commit message: pushing final rev5. may god have mercy.
Parts:
- removed SW1: JS102011SAQN, Button_Switch_SMD:SW_SPDT_CK_JS102011SAQN
- added SW4: JS102011SAQN, Button_Switch_SMD:SW_SPDT_CK_JS102011SAQN, F.Cu at (124.0, 119.0)
- added TP1: TestPoint, TestPoint:TestPoint_Keystone_5015_Micro-Minature, F.Cu at (109.5, 69.0)
- added TP2: TestPoint, TestPoint:TestPoint_Keystone_5015_Micro-Minature, F.Cu at (114.5, 69.0)
- added TP_ADC2: TestPoint, TestPoint:TestPoint_THTPad_D1.5mm_Drill0.7mm, F.Cu at (65.0, 133.5)
- added TP_AND1: TestPoint, TestPoint:TestPoint_THTPad_D1.5mm_Drill0.7mm, F.Cu at (83.5, 107.0)
- added TP_BOOT1: TestPoint, TestPoint:TestPoint_THTPad_D1.5mm_Drill0.7mm, F.Cu at (88.0, 130.0)
- added TP_LCELL_VCC1: TestPoint, TestPoint:TestPoint_THTPad_D1.5mm_Drill0.7mm, F.Cu at (66.0, 149.0)
- added TP_PU_EN1: TestPoint, TestPoint:TestPoint_THTPad_D1.5mm_Drill0.7mm, F.Cu at (108.0, 148.0)
- moved C7 4.23 mm to (81.8, 82.3)
- moved C8 4.23 mm to (84.8, 82.3)
- moved C5 3.99 mm to (72.3, 82.2)
- moved C6 3.99 mm to (76.3, 82.2)
Routing:
- net Net-(J2-Pin_1): track 28.6 -> 39.7 mm
- net GPIO0_BOOT: track 52.3 -> 59.3 mm
- net Net-(R1-Pad1): track 12.7 -> 19.6 mm
- net /controller/ESP_VCC: track 67.2 -> 73.2 mm
- net CHIP_PU_EN: track 65.2 -> 69.7 mm
- net Net-(Q2-E): track 23.3 -> 27.5 mm
- net NFET_3.3V: track 42.5 -> 46.2 mm
- net +5V_WALL: track 123.1 -> 119.9 mm
- net /controller/VBUS: track 39.2 -> 40.3 mm
- net Net-(SW4-C): track 23.1 -> 23.9 mm
- net /controller/USB_D-: track 72.5 -> 73.2 mm
- net +3.3V_WALL: track 58.8 -> 58.2 mm
- net GND: track 0.86 -> 0.76 mm, vias 221 -> 134
Other:
- board text added: "11/21/2024"
- board text removed: "Team 09 FLOPS rev4 11/14/2024"

Commit message: last adds of pdf of sch and pcb
Other:
- board text added: "Load Cell Connect"
Changed lines of the file:
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@@
 	)
 	(gr_rect
-		(start 35 43.5)
-		(end 56 123.5)
+		(start 35.85 59.05)
+		(end 56.85 128.4)
 		(stroke
 			(width 0.1)
@@
 	)
 	(gr_rect
-		(start 77.5 109.5)
-		(end 134 163)
+		(start 77.5 112.45)
+		(end 132.05 163)
 		(stroke
 			(width 0.1)
@@
 	)
 	(gr_rect
-		(start 78 38.5)
-		(end 102 84)
+		(start 82.75 57.7)
+		(end 106.75 103.2)
 		(stroke
 			(width 0.1)
@@
 	)
 	(gr_rect
-		(start 37.5 126)
-		(end 75.5 162.5)
+		(start 37.8 129.55)
+		(end 75.8 160.85)
 		(stroke
 			(width 0.1)
@@
 	)
 	(gr_text "Power FLOPS"
-		(at 81.5 43 0)
+		(at 84.65 61.1 0)
 		(layer "User.1")
 		(effects
@@
 		)
 	)
+	(gr_text "Load Cell Connect"
+		(at 44.35 162.45 0)
+		(layer "User.1")
+		(effects
+			(font
+				(size 1 1)
+				(thickness 0.15)
+			)
+			(justify left bottom)
+		)
+	)
 	(gr_text "Force Sensor Connections"
-		(at 36.5 48.5 0)
-		(layer "User.1")
-		(effects
+		(at 36.45 61.55 0)
+		(layer "User.1")
+		(effects
